Commit message: moveit added

File: biped_description/urdf/control/gazebo_sim_ros2_control.urdf.xacro (robot description, xacro)
@@ -7,5 +7,5 @@
       <!-- IMPORTANT: absolute path avoids find()/env issues -->
       <parameters>
-        /home/vismay/ros2_ws/install/biped_moveit_config/share/biped_moveit_config/config/biped/ros2_controllers.yaml
+        /home/vismay/ros2_ws/install/biped_moveit_config/share/biped_moveit_config/config/biped/biped_controller.yaml
       </parameters>
       <hold_joints>false</hold_joints>

File: biped_description/urdf/robots/biped.xacro (robot description, xacro)
@@ -152,5 +152,5 @@
   <child link="l_hip_link_1"/>
   <axis xyz="0.0 1.0 0.0"/>
-  <dynamics damping="0.01" friction="0.01"/>
+  <dynamics damping="0.01" friction="0.06"/>
 </joint>
 <joint name="l_hip_roll" type="revolute">
@@ -160,5 +160,5 @@
   <child link="l_hip_roll__1"/>
   <axis xyz="-1.0 0.0 0.0"/>
-  <dynamics damping="0.01" friction="0.01"/>
+  <dynamics damping="0.01" friction="0.06"/>
 </joint>
 <joint name="l_knee_roll" type="revolute">
@@ -168,5 +168,5 @@
   <child link="l_knee_link_1"/>
   <axis xyz="-1.0 0.0 0.0"/>
-  <dynamics damping="0.01" friction="0.01"/>
+  <dynamics damping="0.01" friction="0.06"/>
 </joint>
 <joint name="r_abduction" type="revolute">
@@ -176,5 +176,5 @@
   <child link="r_hip_link_1"/>
   <axis xyz="0.0 1.0 0.0"/>
-  <dynamics damping="0.01" friction="0.01"/>
+  <dynamics damping="0.01" friction="0.06"/>
 </joint>
 <joint name="r_hip_roll" type="revolute">
@@ -184,5 +184,5 @@
   <child link="r_hip_roll__1"/>
   <axis xyz="1.0 0.0 0.0"/>
-  <dynamics damping="0.01" friction="0.01"/>
+  <dynamics damping="0.01" friction="0.06"/>
 </joint>
 <joint name="r_knee_roll" type="revolute">
@@ -192,5 +192,5 @@
   <child link="r_knee_link_1"/>
   <axis xyz="1.0 0.0 0.0"/>
-  <dynamics damping="0.01" friction="0.01"/>
+  <dynamics damping="0.01" friction="0.06"/>
 </joint>
 <gazebo reference="l_knee_link_1">

Commit message: Revert "moveit added"
This reverts commit 96171bf940016c9f896ed9cab81dd92a17769e94.

File: biped_description/urdf/control/gazebo_sim_ros2_control.urdf.xacro (robot description, xacro)
@@ -7,5 +7,5 @@
       <!-- IMPORTANT: absolute path avoids find()/env issues -->
       <parameters>
-        /home/vismay/ros2_ws/install/biped_moveit_config/share/biped_moveit_config/config/biped/biped_controller.yaml
+        /home/vismay/ros2_ws/install/biped_moveit_config/share/biped_moveit_config/config/biped/ros2_controllers.yaml
       </parameters>
       <hold_joints>false</hold_joints>

File: biped_description/urdf/robots/biped.xacro (robot description, xacro)
@@ -152,5 +152,5 @@
   <child link="l_hip_link_1"/>
   <axis xyz="0.0 1.0 0.0"/>
-  <dynamics damping="0.01" friction="0.06"/>
+  <dynamics damping="0.01" friction="0.01"/>
 </joint>
 <joint name="l_hip_roll" type="revolute">
@@ -160,5 +160,5 @@
   <child link="l_hip_roll__1"/>
   <axis xyz="-1.0 0.0 0.0"/>
-  <dynamics damping="0.01" friction="0.06"/>
+  <dynamics damping="0.01" friction="0.01"/>
 </joint>
 <joint name="l_knee_roll" type="revolute">
@@ -168,5 +168,5 @@
   <child link="l_knee_link_1"/>
   <axis xyz="-1.0 0.0 0.0"/>
-  <dynamics damping="0.01" friction="0.06"/>
+  <dynamics damping="0.01" friction="0.01"/>
 </joint>
 <joint name="r_abduction" type="revolute">
@@ -176,5 +176,5 @@
   <child link="r_hip_link_1"/>
   <axis xyz="0.0 1.0 0.0"/>
-  <dynamics damping="0.01" friction="0.06"/>
+  <dynamics damping="0.01" friction="0.01"/>
 </joint>
 <joint name="r_hip_roll" type="revolute">
@@ -184,5 +184,5 @@
   <child link="r_hip_roll__1"/>
   <axis xyz="1.0 0.0 0.0"/>
-  <dynamics damping="0.01" friction="0.06"/>
+  <dynamics damping="0.01" friction="0.01"/>
 </joint>
 <joint name="r_knee_roll" type="revolute">
@@ -192,5 +192,5 @@
   <child link="r_knee_link_1"/>
   <axis xyz="1.0 0.0 0.0"/>
-  <dynamics damping="0.01" friction="0.06"/>
+  <dynamics damping="0.01" friction="0.01"/>
 </joint>
 <gazebo reference="l_knee_link_1">
