Commit message: biped setup

File: biped_description/urdf/control/biped_ros2_control.urdf.xacro (robot description, xacro)
@@ -1,13 +1,10 @@
 <?xml version="1.0"?>
 <robot xmlns:xacro="http://www.ros.org/wiki/xacro">
-  <!-- ========================================================= -->
-  <!-- ros2_control hardware specification for BIPED -->
-  <!-- ========================================================= -->
+  <!-- ================= ros2_control ================= -->
   <ros2_control name="BipedSystem" type="system">
-    <!-- Gazebo simulated hardware -->
     <hardware>
       <plugin>gz_ros2_control/GazeboSimSystem</plugin>
     </hardware>
-    <!-- ================= LEFT LEG (ACTUATED) ================= -->
+    <!-- LEFT LEG -->
     <joint name="l_abduction">
       <command_interface name="position"/>
@@ -25,5 +22,10 @@
       <state_interface name="velocity"/>
     </joint>
-    <!-- ================= RIGHT LEG (ACTUATED) ================= -->
+    <joint name="l_foot_roll">
+      <command_interface name="position"/>
+      <state_interface name="position"/>
+      <state_interface name="velocity"/>
+    </joint>
+    <!-- RIGHT LEG -->
     <joint name="r_abduction">
       <command_interface name="position"/>
@@ -41,8 +43,18 @@
       <state_interface name="velocity"/>
     </joint>
-    <!-- ================= PASSIVE JOINTS ================= -->
-    <!-- Feet are intentionally NOT listed -->
-    <!-- left_foot_roll, right_foot_roll -->
-    <!-- Passive joints are handled kinematically -->
+    <joint name="r_foot_roll">
+      <command_interface name="position"/>
+      <state_interface name="position"/>
+      <state_interface name="velocity"/>
+    </joint>
   </ros2_control>
+  <!-- ================= GAZEBO JOINT BINDINGS ================= -->
+  <gazebo reference="l_abduction"><provideFeedback>true</provideFeedback></gazebo>
+  <gazebo reference="l_hip_roll"><provideFeedback>true</provideFeedback></gazebo>
+  <gazebo reference="l_knee_roll"><provideFeedback>true</provideFeedback></gazebo>
+  <gazebo reference="l_foot_roll"><provideFeedback>true</provideFeedback></gazebo>
+  <gazebo reference="r_abduction"><provideFeedback>true</provideFeedback></gazebo>
+  <gazebo reference="r_hip_roll"><provideFeedback>true</provideFeedback></gazebo>
+  <gazebo reference="r_knee_roll"><provideFeedback>true</provideFeedback></gazebo>
+  <gazebo reference="r_foot_roll"><provideFeedback>true</provideFeedback></gazebo>
 </robot>

File: biped_description/urdf/control/gazebo_sim_ros2_control.urdf.xacro (robot description, xacro)
@@ -1,15 +1,13 @@
 <?xml version="1.0"?>
 <robot xmlns:xacro="http://www.ros.org/wiki/xacro">
-<gazebo>
-  <plugin
-    filename="gz_ros2_control-system"
-    name="gz_ros2_control::GazeboSimROS2ControlPlugin">
-    <parameters>
-      $(find biped_moveit_config)/config/biped/ros2_controllers.yaml
-    </parameters>
-    <ros>
-      <remapping>/controller_manager/robot_description:=/robot_description</remapping>
-    </ros>
-  </plugin>
-</gazebo>
+  <gazebo>
+    <plugin
+      filename="gz_ros2_control-system"
+      name="gz_ros2_control::GazeboSimROS2ControlPlugin">
+      <!-- IMPORTANT: absolute path avoids find()/env issues -->
+      <parameters>
+        /home/vismay/ros2_ws/install/biped_moveit_config/share/biped_moveit_config/config/biped/ros2_controllers.yaml
+      </parameters>
+    </plugin>
+  </gazebo>
 </robot>

Commit message: updated robot spawn

File: biped_description/urdf/control/biped_ros2_control.urdf.xacro (robot description, xacro)
@@ -1,10 +1,8 @@
 <?xml version="1.0"?>
 <robot xmlns:xacro="http://www.ros.org/wiki/xacro">
-  <!-- ================= ros2_control ================= -->
   <ros2_control name="BipedSystem" type="system">
     <hardware>
       <plugin>gz_ros2_control/GazeboSimSystem</plugin>
     </hardware>
-    <!-- LEFT LEG -->
     <joint name="l_abduction">
       <command_interface name="position"/>
@@ -22,10 +20,4 @@
       <state_interface name="velocity"/>
     </joint>
-    <joint name="l_foot_roll">
-      <command_interface name="position"/>
-      <state_interface name="position"/>
-      <state_interface name="velocity"/>
-    </joint>
-    <!-- RIGHT LEG -->
     <joint name="r_abduction">
       <command_interface name="position"/>
@@ -43,11 +35,15 @@
       <state_interface name="velocity"/>
     </joint>
+    <joint name="l_foot_roll">
+    <command_interface name="position"/>
+      <state_interface name="position"/>
+      <state_interface name="velocity"/>
+    </joint>
     <joint name="r_foot_roll">
-      <command_interface name="position"/>
+    <command_interface name="position"/>
       <state_interface name="position"/>
       <state_interface name="velocity"/>
     </joint>
   </ros2_control>
-  <!-- ================= GAZEBO JOINT BINDINGS ================= -->
   <gazebo reference="l_abduction"><provideFeedback>true</provideFeedback></gazebo>
   <gazebo reference="l_hip_roll"><provideFeedback>true</provideFeedback></gazebo>

File: biped_description/urdf/robots/biped.xacro (robot description, xacro)
@@ -202,5 +202,5 @@
 </link>
 <joint name="l_abduction" type="revolute">
-  <limit lower="-2.5" upper="0.0" effort="50" velocity="5"/>
+  <limit lower="-2.5" upper="2.5" effort="50" velocity="5"/>
   <origin xyz="-0.05986 -0.04025 -0.0003" rpy="0 0 0"/>
   <parent link="base_link"/>
@@ -210,5 +210,5 @@
 </joint>
 <joint name="l_hip_roll" type="revolute">
-  <limit lower="-2.5" upper="0.0" effort="50" velocity="5"/>
+  <limit lower="-2.5" upper="2.5" effort="50" velocity="5"/>
   <origin xyz="-0.042 0.040277 4.4e-05" rpy="0 0 0"/>
   <parent link="l_hip_link_1"/>
@@ -218,5 +218,5 @@
 </joint>
 <joint name="l_knee_roll" type="revolute">
-  <limit lower="-2.5" upper="0.0" effort="50" velocity="5"/>
+  <limit lower="-2.5" upper="2.5" effort="50" velocity="5"/>
   <origin xyz="-0.047484 0.063923 -0.222186" rpy="0 0 0"/>
   <parent link="l_hip_roll__1"/>
@@ -226,5 +226,5 @@
 </joint>
 <joint name="l_foot_roll" type="revolute">
-  <limit lower="-2.5" upper="0.0" effort="50" velocity="5"/>
+  <limit lower="-2.5" upper="2.5" effort="50" velocity="5"/>
   <origin xyz="-0.02 -0.063862 -0.204573" rpy="0 0 0"/>
   <parent link="l_knee_link_1"/>
@@ -234,5 +234,5 @@
 </joint>
 <joint name="r_abduction" type="revolute">
-  <limit lower="-2.5" upper="0.0" effort="50" velocity="5"/>
+  <limit lower="-2.5" upper="2.5" effort="50" velocity="5"/>
   <origin xyz="-0.00014 -0.04025 -0.0003" rpy="0 0 0"/>
   <parent link="base_link"/>
@@ -242,5 +242,5 @@
 </joint>
 <joint name="r_hip_roll" type="revolute">
-  <limit lower="-2.5" upper="0.0" effort="50" velocity="5"/>
+  <limit lower="-2.5" upper="2.5" effort="50" velocity="5"/>
   <origin xyz="0.042 0.040277 4.4e-05" rpy="0 0 0"/>
   <parent link="r_hip_link_1"/>
@@ -250,5 +250,5 @@
 </joint>
 <joint name="r_knee_roll" type="revolute">
-  <limit lower="-2.5" upper="0.0" effort="50" velocity="5"/>
+  <limit lower="-2.5" upper="2.5" effort="50" velocity="5"/>
   <origin xyz="0.047484 0.063923 -0.222186" rpy="0 0 0"/>
   <parent link="r_hip_roll__1"/>
@@ -258,5 +258,5 @@
 </joint>
 <joint name="r_foot_roll" type="revolute">
-  <limit lower="-2.5" upper="0.0" effort="50" velocity="5"/>
+  <limit lower="-2.5" upper="2.5" effort="50" velocity="5"/>
   <origin xyz="0.02 -0.063862 -0.204573" rpy="0 0 0"/>
   <parent link="r_knee_link_1"/>
@@ -265,3 +265,13 @@
   <dynamics damping="0.5" friction="0.1"/>
 </joint>
+<gazebo reference="base_link">
+  <sensor name="biped_imu" type="imu">
+    <always_on>true</always_on>
+    <update_rate>100</update_rate>
+    <visualize>true</visualize>
+    <topic>imu</topic>
+    <plugin name="gz::sim::systems::Imu" filename="gz-sim-imu-system">
+    </plugin>
+  </sensor>
+</gazebo>
 </robot>
