Commit message: final sorted biped in gazebo-ros

File: biped_description/urdf/robots/biped.xacro (robot description, xacro)
@@ -6,7 +6,13 @@
 <xacro:include filename="$(find biped_description)/urdf/control/biped_ros2_control.urdf.xacro"/>
 <xacro:include filename="$(find biped_description)/urdf/control/gazebo_sim_ros2_control.urdf.xacro"/>
+<link name="base_footprint"/>
+<joint name="base_joint" type="fixed">
+  <parent link="base_footprint"/>
+  <child link="base_link"/>
+  <origin xyz="0 0 0" rpy="0 0 0"/>
+</joint>
 <link name="base_link">
   <inertial>
-    <origin xyz="-0.03000000000000046 -0.05979593496853414 0.004864752592657503" rpy="0 0 0"/>
+    <origin xyz="-0.0300 -0.0597 0.0048" rpy="0 0 0"/>
     <mass value="0.596469253198544"/>
     <inertia ixx="0.000407" iyy="0.001026" izz="0.000804" ixy="0.0" iyz="1.4e-05" ixz="0.0"/>
@@ -22,11 +28,12 @@
     <origin xyz="0 0 0" rpy="0 0 0"/>
     <geometry>
-      <box size="0.05 0.05 0.1"/>
-    </geometry>
+      <mesh filename="file://$(find biped_description)/meshes/biped_280/visual/base_link.stl" scale="0.001 0.001 0.001"/>
+    </geometry>
+    <material name="silver"/>
   </collision>
 </link>
 <link name="l_hip_link_1">
   <inertial>
-    <origin xyz="-0.021972074736058902 0.03692601945677904 3.3809230539884804e-05" rpy="0 0 0"/>
+    <origin xyz="-0.0219 0.0369 3.38e-05" rpy="0 0 0"/>
     <mass value="0.23839991097458857"/>
     <inertia ixx="0.000111" iyy="8.4e-05" izz="0.00011" ixy="1e-05" iyz="0.0" ixz="0.0"/>
@@ -42,11 +49,12 @@
     <origin xyz="0.05986 0.04025 0.0003" rpy="0 0 0"/>
     <geometry>
-      <box size="0.05 0.05 0.1"/>
-    </geometry>
+      <mesh filename="file://$(find biped_description)/meshes/biped_280/visual/l_hip_link_1.stl" scale="0.001 0.001 0.001"/>
+    </geometry>
+    <material name="silver"/>
   </collision>
 </link>
 <link name="l_hip_roll__1">
   <inertial>
-    <origin xyz="-0.02891673482480947 0.031508090951978845 -0.07773431971219692" rpy="0 0 0"/>
+    <origin xyz="-0.0289 0.0315 -0.0777" rpy="0 0 0"/>
     <mass value="0.4778310159751661"/>
     <inertia ixx="0.00221" iyy="0.002059" izz="0.000339" ixy="2.1e-05" iyz="0.000441" ixz="-0.000105"/>
@@ -60,13 +68,14 @@
   </visual>
   <collision>
-    <origin xyz="0.10186 -2.7e-05 0.000256" rpy="0 0 0"/>
-    <geometry>
-      <box size="0.05 0.05 0.1"/>
-    </geometry>
+   <origin xyz="0.10186 -2.7e-05 0.000256" rpy="0 0 0"/>
+    <geometry>
+      <mesh filename="file://$(find biped_description)/meshes/biped_280/visual/l_hip_roll__1.stl" scale="0.001 0.001 0.001"/>
+    </geometry>
+    <material name="silver"/>
   </collision>
 </link>
 <link name="l_knee_link_1">
   <inertial>
-    <origin xyz="-0.019507018919871555 -0.029273752074596843 -0.09345213885570233" rpy="0 0 0"/>
+    <origin xyz="-0.0195 -0.0292 -0.0934" rpy="0 0 0"/>
     <mass value="0.10721414059204377"/>
     <inertia ixx="0.000512" iyy="0.000465" izz="5.9e-05" ixy="-2e-06" iyz="-0.000141" ixz="-5e-06"/>
@@ -82,13 +91,14 @@
     <origin xyz="0.149344 -0.06395 0.222442" rpy="0 0 0"/>
     <geometry>
-     <box size="0.05 0.05 0.1"/>
-    </geometry>
+      <mesh filename="file://$(find biped_description)/meshes/biped_280/visual/l_knee_link_1.stl" scale="0.001 0.001 0.001"/>
+    </geometry>
+    <material name="silver"/>
   </collision>
 </link>
 <link name="l_foot_link__1">
   <inertial>
-    <origin xyz="3.782463971202521e-07 1.2653056471927234e-05 -0.007004050535626083" rpy="0 0 0"/>
+    <origin xyz="0 0.00001 -0.007" rpy="0 0 0"/>
     <mass value="0.01758935163575521"/>
-    <inertia ixx="1.4e-05" iyy="1e-06" izz="1.4e-05" ixy="0.0" iyz="-0.0" ixz="-0.0"/>
+    <inertia ixx="1.4e-05" iyy="1e-06" izz="1.4e-05" ixy="0.0" iyz="0.0" ixz="0.0"/>
   </inertial>
   <visual>
@@ -102,11 +112,12 @@
     <origin xyz="0.169344 -8.8e-05 0.427015" rpy="0 0 0"/>
     <geometry>
-      <box size="0.05 0.05 0.1"/>
-    </geometry>
+      <mesh filename="file://$(find biped_description)/meshes/biped_280/visual/l_foot_link__1.stl" scale="0.001 0.001 0.001"/>
+    </geometry>
+    <material name="silver"/>
   </collision>
 </link>
 <link name="r_hip_link_1">
   <inertial>
-    <origin xyz="0.021972074736058764 0.036926019456778696 3.380923053822375e-05" rpy="0 0 0"/>
+    <origin xyz="0.0219 0.0369 3.38e-05" rpy="0 0 0"/>
     <mass value="0.2383999109745883"/>
     <inertia ixx="0.000111" iyy="8.4e-05" izz="0.00011" ixy="-1e-05" iyz="0.0" ixz="-0.0"/>
@@ -120,13 +131,14 @@
   </visual>
   <collision>
-    <origin xyz="0.00014 0.04025 0.0003" rpy="0 0 0"/>
-    <geometry>
-      <box size="0.05 0.05 0.1"/>
-    </geometry>
+   <origin xyz="0.00014 0.04025 0.0003" rpy="0 0 0"/>
+    <geometry>
+      <mesh filename="file://$(find biped_description)/meshes/biped_280/visual/r_hip_link_1.stl" scale="0.001 0.001 0.001"/>
+    </geometry>
+    <material name="silver"/>
   </collision>
 </link>
 <link name="r_hip_roll__1">
   <inertial>
-    <origin xyz="0.02891673482480684 0.031508090951978915 -0.07773431971220009" rpy="0 0 0"/>
+    <origin xyz="0.0289 0.0315 -0.0777" rpy="0 0 0"/>
     <mass value="0.47783101597516553"/>
     <inertia ixx="0.00221" iyy="0.002059" izz="0.000339" ixy="-2.1e-05" iyz="0.000441" ixz="0.000105"/>
@@ -142,11 +154,12 @@
     <origin xyz="-0.04186 -2.7e-05 0.000256" rpy="0 0 0"/>
     <geometry>
-      <box size="0.05 0.05 0.1"/>
-    </geometry>
+      <mesh filename="file://$(find biped_description)/meshes/biped_280/visual/r_hip_roll__1.stl" scale="0.001 0.001 0.001"/>
+    </geometry>
+    <material name="silver"/>
   </collision>
 </link>
 <link name="r_knee_link_1">
   <inertial>
-    <origin xyz="0.019507018919861743 -0.029273752074596558 -0.09345213885570666" rpy="0 0 0"/>
+    <origin xyz="0.0195 -0.0292 -0.0934" rpy="0 0 0"/>
     <mass value="0.10721414059204377"/>
     <inertia ixx="0.000512" iyy="0.000465" izz="5.9e-05" ixy="2e-06" iyz="-0.000141" ixz="5e-06"/>
@@ -162,13 +175,14 @@
     <origin xyz="-0.089344 -0.06395 0.222442" rpy="0 0 0"/>
     <geometry>
-      <box size="0.05 0.05 0.1"/>
-    </geometry>
+      <mesh filename="file://$(find biped_description)/meshes/biped_280/visual/r_knee_link_1.stl" scale="0.001 0.001 0.001"/>
+    </geometry>
+    <material name="silver"/>
   </collision>
 </link>
 <link name="r_foot_link__1">
   <inertial>
-    <origin xyz="-3.7767476271377554e-07 1.2644456614365469e-05 -0.00700406417380417" rpy="0 0 0"/>
+    <origin xyz="0 0.00001 -0.007" rpy="0 0 0"/>
     <mass value="0.01758928525196201"/>
-    <inertia ixx="1.4e-05" iyy="1e-06" izz="1.4e-05" ixy="-0.0" iyz="-0.0" ixz="0.0"/>
+    <inertia ixx="1.4e-05" iyy="1e-06" izz="1.4e-05" ixy="0.0" iyz="0.0" ixz="0.0"/>
   </inertial>
   <visual>
@@ -182,68 +196,72 @@
     <origin xyz="-0.109344 -8.8e-05 0.427015" rpy="0 0 0"/>
     <geometry>
-      <box size="0.05 0.05 0.1"/>
-    </geometry>
-  </collision>
-</link>
-<joint name="l_abduction" type="continuous">
+      <mesh filename="file://$(find biped_description)/meshes/biped_280/visual/r_foot_link__1.stl" scale="0.001 0.001 0.001"/>
+    </geometry>
+    <material name="silver"/>
+  </collision>
+</link>
+<joint name="l_abduction" type="revolute">
+  <limit lower="-2.5" upper="0.0" effort="50" velocity="5"/>
   <origin xyz="-0.05986 -0.04025 -0.0003" rpy="0 0 0"/>
   <parent link="base_link"/>
   <child link="l_hip_link_1"/>
-  <axis xyz="0.0 1.0 -0.0"/>
-  <dynamics damping="2.0" friction="0.5"/>
-</joint>
-<joint name="l_hip_roll" type="continuous">
+  <axis xyz="0.0 1.0 0.0"/>
+  <dynamics damping="0.5" friction="0.1"/>
+</joint>
+<joint name="l_hip_roll" type="revolute">
+  <limit lower="-2.5" upper="0.0" effort="50" velocity="5"/>
   <origin xyz="-0.042 0.040277 4.4e-05" rpy="0 0 0"/>
   <parent link="l_hip_link_1"/>
   <child link="l_hip_roll__1"/>
-  <axis xyz="-1.0 -0.0 0.0"/>
-  <dynamics damping="2.0" friction="0.5"/>
-</joint>
-<joint name="l_knee_roll" type="continuous">
+  <axis xyz="-1.0 0.0 0.0"/>
+  <dynamics damping="0.5" friction="0.1"/>
+</joint>
+<joint name="l_knee_roll" type="revolute">
+  <limit lower="-2.5" upper="0.0" effort="50" velocity="5"/>
   <origin xyz="-0.047484 0.063923 -0.222186" rpy="0 0 0"/>
   <parent link="l_hip_roll__1"/>
   <child link="l_knee_link_1"/>
-  <axis xyz="-1.0 -0.0 0.0"/>
-  <dynamics damping="2.0" friction="0.5"/>
-</joint>
-<joint name="l_foot_roll" type="continuous">
+  <axis xyz="-1.0 0.0 0.0"/>
+  <dynamics damping="0.5" friction="0.1"/>
+</joint>
+<joint name="l_foot_roll" type="revolute">
+  <limit lower="-2.5" upper="0.0" effort="50" velocity="5"/>
   <origin xyz="-0.02 -0.063862 -0.204573" rpy="0 0 0"/>
   <parent link="l_knee_link_1"/>
   <child link="l_foot_link__1"/>
-  <axis xyz="-1.0 -0.0 0.0"/>
-  <dynamics damping="2.0" friction="0.5"/>
-</joint>
-<joint name="r_abduction" type="continuous">
+  <axis xyz="-1.0 0.0 0.0"/>
+  <dynamics damping="0.5" friction="0.1"/>
+</joint>
+<joint name="r_abduction" type="revolute">
+  <limit lower="-2.5" upper="0.0" effort="50" velocity="5"/>
   <origin xyz="-0.00014 -0.04025 -0.0003" rpy="0 0 0"/>
   <parent link="base_link"/>
   <child link="r_hip_link_1"/>
-  <axis xyz="0.0 1.0 -0.0"/>
-  <dynamics damping="2.0" friction="0.5"/>
-</joint>
-<joint name="r_hip_roll" type="continuous">
+  <axis xyz="0.0 1.0 0.0"/>
+  <dynamics damping="0.5" friction="0.1"/>
+</joint>
+<joint name="r_hip_roll" type="revolute">
+  <limit lower="-2.5" upper="0.0" effort="50" velocity="5"/>
   <origin xyz="0.042 0.040277 4.4e-05" rpy="0 0 0"/>
   <parent link="r_hip_link_1"/>
   <child link="r_hip_roll__1"/>
-  <axis xyz="1.0 -0.0 -0.0"/>
-  <dynamics damping="2.0" friction="0.5"/>
-</joint>
-<joint name="r_knee_roll" type="continuous">
+  <axis xyz="1.0 0.0 0.0"/>
+  <dynamics damping="0.5" friction="0.1"/>
+</joint>
+<joint name="r_knee_roll" type="revolute">
+  <limit lower="-2.5" upper="0.0" effort="50" velocity="5"/>
   <origin xyz="0.047484 0.063923 -0.222186" rpy="0 0 0"/>
   <parent link="r_hip_roll__1"/>
   <child link="r_knee_link_1"/>
-  <axis xyz="1.0 0.0 -0.0"/>
-  <dynamics damping="2.0" friction="0.5"/>
-</joint>
-<joint name="r_foot_roll" type="continuous">
+  <axis xyz="1.0 0.0 0.0"/>
+  <dynamics damping="0.5" friction="0.1"/>
+</joint>
+<joint name="r_foot_roll" type="revolute">
+  <limit lower="-2.5" upper="0.0" effort="50" velocity="5"/>
   <origin xyz="0.02 -0.063862 -0.204573" rpy="0 0 0"/>
   <parent link="r_knee_link_1"/>
   <child link="r_foot_link__1"/>
-  <axis xyz="-1.0 -0.0 0.0"/>
-  <dynamics damping="2.0" friction="0.5"/>
-</joint>
-<link name="world"/>
-<joint name="world_to_base" type="fixed">
-  <parent link="world"/>
-  <child link="base_link"/>
+  <axis xyz="-1.0 0.0 0.0"/>
+  <dynamics damping="0.5" friction="0.1"/>
 </joint>
 </robot>

Commit message: push test

File: biped_description/urdf/robots/biped.xacro (robot description, xacro)
@@ -152,5 +152,5 @@
   <child link="l_hip_link_1"/>
   <axis xyz="0.0 1.0 0.0"/>
-  <dynamics damping="0.5" friction="0.1"/>
+  <dynamics damping="0.01" friction="0.01"/>
 </joint>
 <joint name="l_hip_roll" type="revolute">
@@ -160,5 +160,5 @@
   <child link="l_hip_roll__1"/>
   <axis xyz="-1.0 0.0 0.0"/>
-  <dynamics damping="0.5" friction="0.1"/>
+  <dynamics damping="0.01" friction="0.01"/>
 </joint>
 <joint name="l_knee_roll" type="revolute">
@@ -168,5 +168,5 @@
   <child link="l_knee_link_1"/>
   <axis xyz="-1.0 0.0 0.0"/>
-  <dynamics damping="0.5" friction="0.1"/>
+  <dynamics damping="0.01" friction="0.01"/>
 </joint>
 <joint name="r_abduction" type="revolute">
@@ -176,5 +176,5 @@
   <child link="r_hip_link_1"/>
   <axis xyz="0.0 1.0 0.0"/>
-  <dynamics damping="0.5" friction="0.1"/>
+  <dynamics damping="0.01" friction="0.01"/>
 </joint>
 <joint name="r_hip_roll" type="revolute">
@@ -184,5 +184,5 @@
   <child link="r_hip_roll__1"/>
   <axis xyz="1.0 0.0 0.0"/>
-  <dynamics damping="0.5" friction="0.1"/>
+  <dynamics damping="0.01" friction="0.01"/>
 </joint>
 <joint name="r_knee_roll" type="revolute">
@@ -192,17 +192,21 @@
   <child link="r_knee_link_1"/>
   <axis xyz="1.0 0.0 0.0"/>
-  <dynamics damping="0.5" friction="0.1"/>
-</joint>
-<gazebo reference="l_foot_link__1">
-  <mu1>0.6</mu1>
-  <mu2>0.6</mu2>
-  <kp>500000</kp>     <!-- contact stiffness -->
-  <kd>2000</kd>       <!-- contact damping -->
+  <dynamics damping="0.01" friction="0.01"/>
+</joint>
+<gazebo reference="l_knee_link_1">
+  <mu1>0.9</mu1>
+  <mu2>0.9</mu2>
+  <kp>100000.0</kp>
+  <kd>1.0</kd>
+  <minDepth>0.001</minDepth>
+  <maxVel>0.1</maxVel>
 </gazebo>
-<gazebo reference="r_foot_link__1">
-  <mu1>0.6</mu1>
-  <mu2>0.6</mu2>
-  <kp>500000</kp>
-  <kd>2000</kd>
+<gazebo reference="r_knee_link_1">
+  <mu1>0.9</mu1>
+  <mu2>0.9</mu2>
+  <kp>100000.0</kp>
+  <kd>1.0</kd>
+  <minDepth>0.001</minDepth>
+  <maxVel>0.1</maxVel>
 </gazebo>
 <gazebo reference="base_link">

Commit message: corrected imu and added a shit IK walker script

File: biped_description/urdf/robots/biped.xacro (robot description, xacro)
@@ -210,5 +210,18 @@
   <maxVel>0.1</maxVel>
 </gazebo>
-<gazebo reference="base_link">
+<link name="imu_link">
+  <inertial>
+    <mass value="0.001"/>
+    <origin xyz="0 0 0" rpy="0 0 0"/>
+    <inertia ixx="1e-06" iyy="1e-06" izz="1e-06" ixy="0" iyz="0" ixz="0"/>
+  </inertial>
+</link>
+<joint name="imu_joint" type="fixed">
+  <parent link="base_link"/>
+  <child link="imu_link"/>
+  <origin xyz="0 0 0" rpy="0 0 0"/>
+</joint>
+<gazebo reference="imu_link">
+  <gravity>true</gravity>
   <sensor name="biped_imu" type="imu">
     <always_on>true</always_on>
